File: clock/clock.kicad_sch (KiCad schematic)
At the start: 80 parts, among them J1 IN-12, J2 IN-12, J3 IN-12, J4 IN-12, J5 USB_C_Receptacle_USB2.0_14P, Q1 MMBTA42, Q10 MMBTA42, Q11 MMBTA42, Q12 MMBTA42, Q13 PMOS, Q14 MMBTA42, Q15 PMOS, Q16 MMBTA42, Q17 PMOS, Q18 MMBTA42, Q2 PMOS, Q3 MMBTA42, Q4 MMBTA42, Q5 MMBTA42, Q6 MMBTA42, Q7 MMBTA42, Q8 MMBTA42, Q9 MMBTA42, SW1 SW_Push, SW2 SW_Push, U1 RP2040, U2 AP2112K-3.3TRG1, U3 PCF8563T, Y1 ABM8-272-T3, Y2 Seiko SC-32S（LCSC C97604）

Commit message: LD2410S add
Parts:
- added C6: 1uF, Capacitor_SMD:C_0603_1608Metric, symbol Device:C
- added J6, J7: Conn_01x04_Pin, Connector_PinSocket_2.54mm:PinSocket_1x04_P2.54mm_Vertical, symbol Connector:Conn_01x04_Pin
- added J8: Debug_pin, Connector_PinSocket_2.54mm:PinSocket_1x04_P2.54mm_Horizontal, symbol Connector:Conn_01x04_Pin
- added J9: LD2410S, symbol Connector:Conn_01x05_Pin
- added U4: W25Q16JV, Package_SO:SOIC-8_5.3x5.3mm_P1.27mm, symbol Memory_Flash:W25Q16JVSS
- C1, C2, C3, C4, C5: footprint (none) -> Capacitor_SMD:C_0603_1608Metric
- D1: value BAS70-04 -> BAS70-05
- J5: footprint (none) -> Connector_USB:USB_C_Receptacle_Palconn_UTC16-G
- Q13, Q15, Q17, Q2: footprint (none) -> Package_TO_SOT_SMD:SC-59
- R1, R10, R11, R12, R13, R14, R15, R16, R17, R18, R19, R2, R20, R21, R22, R23, R24, R25, R26, R27, R28, R29, R3, R30, R31, R32, R33, R34, R35, R36, R37, R38, R39, R4, R40, R41, R42, R43, R5, R6, R7, R8, R9: footprint (none) -> Resistor_SMD:R_0603_1608Metric
- SW1: value SW_Push -> RESET_SW
- SW2: value SW_Push -> BOOTSEL_SW
- Y1: footprint (none) -> Crystal:Crystal_SMD_0603-4Pin_6.0x3.5mm
- Y2: footprint (none) -> Crystal:Crystal_AT310_D3.0mm_L10.0mm_Horizontal
Connections:
- net 170V: now also J7.3 (Pin_3)
- net 3.3V: now also C6.2, J9.1 (Pin_1), U4.8 (VCC)
- net 5V: now also J7.1 (Pin_1)
- net GND: now also U1.19 (TESTEN), C6.1, J6.4 (Pin_4), J7.2 (Pin_2), J7.4 (Pin_4), J8.4 (Pin_4), J9.2 (Pin_2), U4.4 (GND)
- net GPS_RX: now also J6.3 (Pin_3)
- net GPS_TX: now also J6.2 (Pin_2)
- net at R41.1, U1.56 (~{QSPI_SS}): now also U4.1 (~{CS})
- net at U1.24 (SWCLK): now also J8.2 (Pin_2)
- net at U1.25 (SWDIO): now also J8.3 (Pin_3)
- net LD2410S_RX: now reaches U1.31 (GPIO20)
- net LD2410S_RX: now also J9.4 (Pin_4)
- net LD2410S_OT1: now reaches U1.32 (GPIO21)
- net LD2410S_OT1: now also J9.3 (Pin_3)
- net LD2410S_OT2: now reaches U1.34 (GPIO22)
- net LD2410S_OT2: now also J9.5 (Pin_5)
- net at U1.51 (QSPI_SD3): now also U4.7 (~{HOLD}/~{RESET}/IO_{3})
- net at U1.52 (QSPI_SCLK): now also U4.6 (CLK)
- net at U1.53 (QSPI_SD0): now also U4.5 (DI/IO_{0})
- net at U1.54 (QSPI_SD2): now also U4.3 (~{WP}/IO_{2})
- net at U1.55 (QSPI_SD1): now also U4.2 (DO/IO_{1})
- new net VCC: J6.1 (Pin_1), J8.1 (Pin_1)
- no-connect marks 2 -> 11
Other:
- note added: "170V Power Supply"
- note added: "3.3V Power Supply"
- note added: "GNSS PIN"
- note added: "LD2410S PIN"
- note added: "Nixie Tube Controller"
- note added: "RP2040 & ROM"
- note added: "RTC & Battery"
- note added: "USB C Connector"
- moved on the sheet: BT1, C1, C2, C3, C4, C5, D1, J1, J2, J3, J4, Q1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

Commit message: 調整: 回路図の部品位置とワイヤーを修正
Connections:
- net GPS_RX: now also U1.2 (GPIO0); no longer U1.3 (GPIO1)
- net GPS_TX: now also U1.3 (GPIO1); no longer U1.2 (GPIO0)
Other:
- moved on the sheet: J5, R37, R38, R39, R40
